File: BUTTON_OPENER/BUTTON_OPENER.kicad_sch (KiCad schematic)
At the start: 68 parts, among them J1 N/A, J2 OPTO_OUT_1, J3 OPTO_OUT_2, J4 OPTO_IN_1, J5 OPTO_IN_2, J6 Conn_01x05, P1 USB_C_Plug_USB2.0, Q1 BC847, Q2 BC847, SW1 N/A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

Commit message: Updated HW
Parts:
- D1, U2, U8: now left out of the parts list
Connections:
- net EN: now also U2.26 (IO4); no longer U2.9 (IO33)
- net OPTO_IN1: now also U2.9 (IO33); no longer U2.26 (IO4)
- net at U5.3: now also J3.2 (Pin_2); no longer J3.1 (Pin_1)
- net at U5.4: now also J3.1 (Pin_1); no longer J3.2 (Pin_2)
- net at J2.1 (Pin_1): now also U4.4; no longer U4.3
- net at J2.2 (Pin_2): now also U4.3; no longer U4.4
Other:
- moved on the sheet: J2, J3
Changed lines of the file:
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@@
 	)
 	(label "EN"
-		(at 170.18 104.14 0)
+		(at 170.18 60.96 0)
 		(effects
 			(font
@@
 	)
 	(label "OPTO_IN1"
-		(at 170.18 60.96 0)
+		(at 170.18 104.14 0)
 		(effects
 			(font
@@
 	(symbol
 		(lib_id "Connector:Conn_01x02_Pin")
-		(at 270.51 102.87 180)
+		(at 270.51 100.33 0)
+		(mirror y)
 		(unit 1)
 		(exclude_from_sim no)
@@
 		(on_board yes)
 		(dnp no)
-		(fields_autoplaced yes)
 		(property "Reference" "J2"
-			(at 271.78 100.3299 0)
+			(at 271.78 102.8701 0)
 			(effects
 				(font
@@
 		)
 		(property "Value" "OPTO_OUT_1"
-			(at 271.78 102.8699 0)
+			(at 271.78 100.3301 0)
 			(effects
 				(font
@@
 		)
 		(property "Footprint" "Connector_Phoenix_MC:PhoenixContact_MCV_1,5_2-G-3.5_1x02_P3.50mm_Vertical"
-			(at 270.51 102.87 0)
+			(at 270.51 100.33 0)
 			(effects
 				(font
@@
 		)
 		(property "Datasheet" "~"
-			(at 270.51 102.87 0)
+			(at 270.51 100.33 0)
 			(effects
 				(font
@@
 		)
 		(property "Description" "Generic connector, single row, 01x02, script generated"
-			(at 270.51 102.87 0)
+			(at 270.51 100.33 0)
 			(effects
 				(font
@@
 		)
 		(property "tolerance" ""
-			(at 270.51 102.87 0)
+			(at 270.51 100.33 0)
 			(effects
 				(font
@@
 		)
 		(property "type" ""
-			(at 270.51 102.87 0)
+			(at 270.51 100.33 0)
 			(effects
 				(font
@@
 		)
 		(property "voltage" ""
-			(at 270.51 102.87 0)
+			(at 270.51 100.33 0)
 			(effects
 				(font
@@
 		(unit 1)
 		(exclude_from_sim no)
-		(in_bom yes)
+		(in_bom no)
 		(on_board yes)
 		(dnp no)
@@
 	(symbol
 		(lib_id "Connector:Conn_01x02_Pin")
-		(at 270.51 116.84 180)
+		(at 270.51 114.3 0)
+		(mirror y)
 		(unit 1)
 		(exclude_from_sim no)
@@
 		(on_board yes)
 		(dnp no)
-		(fields_autoplaced yes)
 		(property "Reference" "J3"
-			(at 271.78 114.2999 0)
+			(at 271.78 116.8401 0)
 			(effects
 				(font
@@
 		)
 		(property "Value" "OPTO_OUT_2"
-			(at 271.78 116.8399 0)
+			(at 271.78 114.3001 0)
 			(effects
 				(font
@@
 		)
 		(property "Footprint" "Connector_Phoenix_MC:PhoenixContact_MCV_1,5_2-G-3.5_1x02_P3.50mm_Vertical"
-			(at 270.51 116.84 0)
+			(at 270.51 114.3 0)
 			(effects
 				(font
@@
 		)
 		(property "Datasheet" "~"
-			(at 270.51 116.84 0)
+			(at 270.51 114.3 0)
 			(effects
 				(font
@@
 		)
 		(property "Description" "Generic connector, single row, 01x02, script generated"
-			(at 270.51 116.84 0)
+			(at 270.51 114.3 0)
 			(effects
 				(font
@@
 		)
 		(property "tolerance" ""
-			(at 270.51 116.84 0)
+			(at 270.51 114.3 0)
 			(effects
 				(font
@@
 		)
 		(property "type" ""
-			(at 270.51 116.84 0)
+			(at 270.51 114.3 0)
 			(effects
 				(font
@@
 		)
 		(property "voltage" ""
-			(at 270.51 116.84 0)
+			(at 270.51 114.3 0)
 			(effects
 				(font
@@
 		(unit 1)
 		(exclude_from_sim no)
-		(in_bom yes)
+		(in_bom no)
 		(on_board yes)
 		(dnp no)
@@
 		(unit 1)
 		(exclude_from_sim no)
-		(in_bom yes)
+		(in_bom no)
 		(on_board yes)
 		(dnp no)

Commit message: Update
Connectors to screw terminals
Regulator to low dropout buck
USB C CC Resistors
IO2 pulldown resistor added
Parts:
- removed C20, C3: 10uF, Capacitor_SMD:C_0603_1608Metric, symbol Device:C
- removed J2: OPTO_OUT_1, Connector_Phoenix_MC:PhoenixContact_MCV_1,5_2-G-3.5_1x02_P3.50mm_Vertical, symbol Connector:Conn_01x02_Pin
- removed J3: OPTO_OUT_2, Connector_Phoenix_MC:PhoenixContact_MCV_1,5_2-G-3.5_1x02_P3.50mm_Vertical, symbol Connector:Conn_01x02_Pin
- removed J4: OPTO_IN_1, Connector_Phoenix_MC:PhoenixContact_MCV_1,5_2-G-3.5_1x02_P3.50mm_Vertical, symbol Connector:Conn_01x02_Pin
- removed J5: OPTO_IN_2, Connector_Phoenix_MC:PhoenixContact_MCV_1,5_2-G-3.5_1x02_P3.50mm_Vertical, symbol Connector:Conn_01x02_Pin
- removed P1: USB_C_Plug_USB2.0, Connector_USB:USB_C_Receptacle_GCT_USB4105-xx-A_16P_TopMnt_Horizontal, symbol Connector:USB_C_Plug_USB2.0
- removed U1: N/A, Package_TO_SOT_SMD:SOT-223-3_TabPin2, symbol Regulator_Linear:AMS1117-3.3
- added J2, J3: Screw_Terminal_01x04, TerminalBlock:TerminalBlock_MaiXu_MX126-5.0-04P_1x04_P5.00mm, symbol Connector:Screw_Terminal_01x04
- added J7: USB_C_Receptacle_USB2.0_14P, Connector_USB:USB_C_Receptacle_G-Switch_GT-USB-7010ASV, symbol Connector:USB_C_Receptacle_USB2.0_14P
- added R34, R35: 5.1k, Resistor_SMD:R_0603_1608Metric, symbol Device:R
- SW1, SW2: now left out of the parts list
- U2: value N/A -> ESP32-WROOM
- U8: value N/A -> CP2102N
Connections:
- net +3V3: no longer R9.1
- net CHRG: now also U2.16 (IO13); no longer U2.37 (IO23)
- net D+: now also J7.A6 (D+), J7.B6 (D+)
- net D-: now also J7.A7 (D-), J7.B7 (D-)
- net GND: now also R9.2, J7.A1 (GND), J7.A12 (GND), J7.B1 (GND), J7.B12 (GND), J7.S1 (SHIELD), R34.1, R35.1
- net STDBY: now also U2.37 (IO23); no longer U2.16 (IO13)
- net VBUS: now also J7.A4 (VBUS), J7.A9 (VBUS), J7.B4 (VBUS), J7.B9 (VBUS)
- net at U5.3: now also J2.1 (Pin_1)
- net at U5.4: now also J2.2 (Pin_2)
- net at D3.2 (A): now also J3.3 (Pin_3)
- net at U4.4: now also J2.4 (Pin_4)
- net at U4.3: now also J2.3 (Pin_3)
- net at C14.2, U7.2: now also J3.4 (Pin_4)
- net at U2.14 (IO12): now also R9.1
- net at U2.23 (IO15): no longer R9.2
- net at C12.2, U6.2: now also J3.2 (Pin_2)
- net at D2.2 (A): now also J3.1 (Pin_1)
- new net: J7.B5 (CC2), R34.2
- new net: J7.A5 (CC1), R35.2
- no-connect marks 12 -> 9
Other:
- added sheet buck (buck.kicad_sch)
- moved on the sheet: R9

Commit message: PCB ordered with this commit
Parts:
- added H1, H2, H3, H4: MountingHole, MountingHole:MountingHole_3.2mm_M3, symbol Mechanical:MountingHole
- C1: JLCPCB Part # (none) -> C19702
- C10, C11, C12, C13, C14, C15, C17, C4, C7, C8: JLCPCB Part # (none) -> C14663
- C16, C9: JLCPCB Part # (none) -> C19666
- C2: JLCPCB Part # (none) -> C106248
- C5, C6: value N/A -> 100nF; JLCPCB Part # (none) -> C14663
- D2, D3, D4, J1, J2, J3, J6: now not fitted; now left out of the parts list
- J7: JLCPCB Part # (none) -> C2927039
- Q1, Q2: JLCPCB Part # (none) -> C475630
- R1: JLCPCB Part # (none) -> C25804
- R10: value 1k -> 1K5; JLCPCB Part # (none) -> C22843
- R11, R12: value 3k3 -> 3K3; JLCPCB Part # (none) -> C22978
- R13, R15, R16, R21, R25, R8: value 1k -> 1K; JLCPCB Part # (none) -> C21190
- R14, R19, R24: JLCPCB Part # (none) -> C25819
- R17, R2, R3, R9: JLCPCB Part # (none) -> C4216
- R18: JLCPCB Part # (none) -> C21190
- R20: value 1k -> 8K2; JLCPCB Part # (none) -> C25981
- R22, R26: value 10k -> 10K; JLCPCB Part # (none) -> C25804
- R23, R27: JLCPCB Part # (none) -> C22790
- R34, R35: value 5.1k -> 5K1; JLCPCB Part # (none) -> C23186
- R4, R5: value N/A -> 6K8; JLCPCB Part # (none) -> C23212
- R6, R7: value N/A -> 1K; JLCPCB Part # (none) -> C21190
- SW1, SW2, U2: now not fitted
- U3: JLCPCB Part # (none) -> C31810
- U4, U5, U6, U7: JLCPCB Part # (none) -> C123196
- U8: JLCPCB Part # (none) -> C969151; now in the parts list
