File: BUTTON_OPENER/battery.kicad_sch (KiCad schematic)
At the start: 12 parts, among them Q3 BSD840N, U10 TP4056-42-ESOP8, U9 DW01A

Commit message: PCB ordered with this commit
Parts:
- BT1: now not fitted; now left out of the parts list
- C18, C19: JLCPCB Part # (none) -> C14663
- Q3: JLCPCB Part # (none) -> C466988
- R28: JLCPCB Part # (none) -> C22775
- R29, R30: value N/A -> 47K; now not fitted; now left out of the parts list
- R31: value N/A -> 0R; JLCPCB Part # (none) -> C21189
- R32: value 1k -> 1K; JLCPCB Part # (none) -> C21190
- R33: value 2k2 -> 2K2; JLCPCB Part # (none) -> C4190
- U10: JLCPCB Part # (none) -> C16581
- U9: JLCPCB Part # (none) -> C2927799
Changed lines of the file:
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@@
+			)
+		)
+		(property "JLCPCB Part #" "C466988"
+			(at 190.5 111.76 90)
+			(effects
+				(font
+					(size 1.27 1.27)
+				)
+				(hide yes)
 			)
 		)
@@
 			)
 		)
+		(property "JLCPCB Part #" "C466988"
+			(at 172.72 111.76 90)
+			(effects
+				(font
+					(size 1.27 1.27)
+				)
+				(hide yes)
+			)
+		)
 		(pin "6"
 		)
@@
 			)
 		)
-		(property "Value" "2k2"
+		(property "Value" "2K2"
 			(at 137.16 121.9199 0)
 			(effects
@@
 		)
 		(property "voltage" ""
+			(at 134.62 120.65 0)
+			(effects
+				(font
+					(size 1.27 1.27)
+				)
+				(hide yes)
+			)
+		)
+		(property "JLCPCB Part #" "C4190"
 			(at 134.62 120.65 0)
 			(effects
@@
 			)
 		)
+		(property "JLCPCB Part #" "C16581"
+			(at 119.38 111.76 0)
+			(effects
+				(font
+					(size 1.27 1.27)
+				)
+				(hide yes)
+			)
+		)
 		(pin "8"
 		)
@@
 			)
 		)
-		(property "Value" "N/A"
+		(property "Value" "0R"
 			(at 105.41 101.5999 0)
 			(effects
@@
 		)
 		(property "voltage" ""
+			(at 102.87 100.33 0)
+			(effects
+				(font
+					(size 1.27 1.27)
+				)
+				(hide yes)
+			)
+		)
+		(property "JLCPCB Part #" "C21189"
 			(at 102.87 100.33 0)
 			(effects
@@
 			)
 		)
-		(property "Value" "1k"
+		(property "Value" "1K"
 			(at 201.93 101.5999 0)
 			(effects
@@
 		)
 		(property "voltage" ""
+			(at 199.39 100.33 0)
+			(effects
+				(font
+					(size 1.27 1.27)
+				)
+				(hide yes)
+			)
+		)
+		(property "JLCPCB Part #" "C21190"
 			(at 199.39 100.33 0)
 			(effects
@@
 		(unit 1)
 		(exclude_from_sim no)
-		(in_bom yes)
+		(in_bom no)
 		(on_board yes)
-		(dnp no)
+		(dnp yes)
 		(fields_autoplaced yes)
 		(property "Reference" "BT1"
@@
 		)
 		(property "voltage" ""
+			(at 213.36 95.25 0)
+			(effects
+				(font
+					(size 1.27 1.27)
+				)
+				(hide yes)
+			)
+		)
+		(property "JLCPCB Part #" ""
 			(at 213.36 95.25 0)
 			(effects
@@
 		)
 		(property "voltage" ""
+			(at 161.29 91.44 0)
+			(effects
+				(font
+					(size 1.27 1.27)
+				)
+				(hide yes)
+			)
+		)
+		(property "JLCPCB Part #" "C14663"
 			(at 161.29 91.44 0)
 			(effects
@@
 			)
 		)
+		(property "JLCPCB Part #" "C2927799"
+			(at 182.88 88.9 0)
+			(effects
+				(font
+					(size 1.27 1.27)
+				)
+				(hide yes)
+			)
+		)
 		(pin "4"
 		)
@@
 		(unit 1)
 		(exclude_from_sim no)
-		(in_bom yes)
+		(in_bom no)
 		(on_board yes)
-		(dnp no)
+		(dnp yes)
 		(fields_autoplaced yes)
 		(property "Reference" "R30"
@@
 			)
 		)
-		(property "Value" "N/A"
+		(property "Value" "47K"
 			(at 92.71 101.5999 0)
 			(effects
@@
 		)
 		(property "voltage" ""
+			(at 90.17 100.33 0)
+			(effects
+				(font
+					(size 1.27 1.27)
+				)
+				(hide yes)
+			)
+		)
+		(property "JLCPCB Part #" ""
 			(at 90.17 100.33 0)
 			(effects
@@
 			)
 		)
+		(property "JLCPCB Part #" "C22775"
+			(at 152.4 86.36 90)
+			(effects
+				(font
+					(size 1.27 1.27)
+				)
+				(hide yes)
+			)
+		)
 		(pin "2"
 		)
@@
 		(unit 1)
 		(exclude_from_sim no)
-		(in_bom yes)
+		(in_bom no)
 		(on_board yes)
-		(dnp no)
+		(dnp yes)
 		(fields_autoplaced yes)
 		(property "Reference" "R29"
@@
 			)
 		)
-		(property "Value" "N/A"
+		(property "Value" "47K"
 			(at 83.82 101.5999 0)
 			(effects
@@
 		)
 		(property "voltage" ""
+			(at 81.28 100.33 0)
+			(effects
+				(font
+					(size 1.27 1.27)
+				)
+				(hide yes)
+			)
+		)
+		(property "JLCPCB Part #" ""
 			(at 81.28 100.33 0)
 			(effects
@@
 			(at 111.76 96.52 0)
 			(effects
+				(font
+					(size 1.27 1.27)
+				)
+				(hide yes)
+			)
+		)
+		(property "JLCPCB Part #" "C14663"
+			(at 111.76 96.52 0)
+			(effects
