File: BUTTON_OPENER/buck.kicad_sch (KiCad schematic)
At the start: 7 parts, among them U11 TLV62568DBV

Commit message: PCB ordered with this commit
Parts:
- C20, C3: value 10uF 6.3V X7R -> 10uF; JLCPCB Part # (none) -> C19702
- C21: value NC -> 22pF
- L1: footprint Inductor_SMD:L_APV_ANR4020 -> Inductor_SMD:L_APV_ANR4026; JLCPCB Part # (none) -> C167854
- R36: now not fitted; now left out of the parts list
- R37: JLCPCB Part # (none) -> C25808
- U11: value TLV62568DBV -> SUNTEK SK6615CS5; JLCPCB Part # (none) -> C2986199
Changed lines of the file:
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@@
 			)
 		)
-		(property "Value" "10uF 6.3V X7R"
+		(property "Value" "10uF"
 			(at 167.64 87.6299 0)
 			(effects
@@
 		)
 		(property "voltage" ""
+			(at 163.83 86.36 0)
+			(effects
+				(font
+					(size 1.27 1.27)
+				)
+				(hide yes)
+			)
+		)
+		(property "JLCPCB Part #" "C19702"
 			(at 163.83 86.36 0)
 			(effects
@@
 		(unit 1)
 		(exclude_from_sim no)
-		(in_bom yes)
+		(in_bom no)
 		(on_board yes)
-		(dnp no)
+		(dnp yes)
 		(property "Reference" "R36"
 			(at 147.32 81.28 90)
@@
 		)
 		(property "voltage" ""
+			(at 147.32 81.28 90)
+			(effects
+				(font
+					(size 1.27 1.27)
+				)
+				(hide yes)
+			)
+		)
+		(property "JLCPCB Part #" ""
 			(at 147.32 81.28 90)
 			(effects
@@
 			)
 		)
-		(property "Value" "NC"
+		(property "Value" "22pF"
 			(at 157.48 82.5499 0)
 			(effects
@@
 		)
 		(property "voltage" ""
+			(at 153.67 81.28 0)
+			(effects
+				(font
+					(size 1.27 1.27)
+				)
+				(hide yes)
+			)
+		)
+		(property "JLCPCB Part #" ""
 			(at 153.67 81.28 0)
 			(effects
@@
 			)
 		)
+		(property "JLCPCB Part #" "C25808"
+			(at 147.32 91.44 90)
+			(effects
+				(font
+					(size 1.27 1.27)
+				)
+				(hide yes)
+			)
+		)
 		(pin "2"
 		)
@@
 			)
 		)
-		(property "Value" "10uF 6.3V X7R"
+		(property "Value" "10uF"
 			(at 100.33 87.6299 0)
 			(effects
@@
 		)
 		(property "voltage" ""
+			(at 96.52 86.36 0)
+			(effects
+				(font
+					(size 1.27 1.27)
+				)
+				(hide yes)
+			)
+		)
+		(property "JLCPCB Part #" "C19702"
 			(at 96.52 86.36 0)
 			(effects
@@
 			)
 		)
-		(property "Value" "TLV62568DBV"
+		(property "Value" "SUNTEK  SK6615CS5"
 			(at 123.19 71.12 0)
 			(effects
@@
 			)
 		)
-		(property "Datasheet" "http://www.ti.com/lit/ds/symlink/tlv62568.pdf"
+		(property "Datasheet" "https://jlcpcb.com/api/file/downloadByFileSystemAccessId/8590910237937651712"
 			(at 116.84 67.31 0)
 			(effects
@@
 			)
 		)
-		(property "Description" "High Efficiency Synchronous Buck Converter, Adjustable Output 0.6V-5.5V, 1A, SOT-23-5"
+		(property "Description" ""
+			(at 123.19 78.74 0)
+			(effects
+				(font
+					(size 1.27 1.27)
+				)
+				(hide yes)
+			)
+		)
+		(property "JLCPCB Part #" "C2986199"
 			(at 123.19 78.74 0)
 			(effects
@@
 			)
 		)
-		(property "Footprint" "Inductor_SMD:L_APV_ANR4020"
+		(property "Footprint" "Inductor_SMD:L_APV_ANR4026"
 			(at 139.7 76.2 0)
 			(effects
@@
 			(effects
 				(font
+					(size 1.27 1.27)
+				)
+				(hide yes)
+			)
+		)
+		(property "JLCPCB Part #" "C167854"
+			(at 139.7 76.2 90)
+			(effects
+				(font
